File: LED-Square_PT4115.kicad_pcb (KiCad board)
At the start: 2 copper layers, 50 x 50 mm, 30 parts, among them P1 IN, P2 OUT, U1 PT4115-SOT89-5

Commit message: Adapted to changed footprint 'MADW__edge-connector_SIL6_female'.
Parts:
- P1: footprint MADW__edge-connector_SIL6_female -> my_parts:MADW__edge-connector_SIL6_female
Other:
- board text added: "LED Square V1.11.f"
- board text removed: "LED Square V1.11.e"

Commit message: Now using 2 pins for the DIM signal as well.
Parts:
- L1: footprint -L1812 -> my_parts:MADW__L4.8x3.3mm
- renumbered G*** to G3, G*** to G4
Connections:
- P1 pad 5: Net-(P1-Pad5) -> /DIM
- P2 pad 2: Net-(P2-Pad2) -> /DIM
Routing:
- net /DIM: track 50.9 -> 56.0 mm
Other:
- board text added: "LED Square V1.2.a"
- board text removed: "LED Square V1.11.f"
- board text removed: "NC"
