File: LED-Square_PT4115.sch (KiCad schematic (older format))
At the start: 25 parts, among them P1 IN, P2 OUT, U1 PT4115-SOT89-5

Commit message: Prototype worked well with 1k + 5V1 Zener, so switched to that.
Parts:
- DZ1: value BZX84C_5V6 -> BZX84C_5V1
Changed lines of the file:
@@
-EESchema Schematic File Version 2  date Sun 18 Nov 2012 06:39:24 PM CET
+EESchema Schematic File Version 2  date Tue 20 Nov 2012 04:58:50 PM CET
 LIBS:my_parts
 LIBS:power
@@
 Sheet 1 1
 Title "LED-Square PT4115"
-Date "13 nov 2012"
+Date "20 nov 2012"
 Rev "1.0"
 Comp "2012 - blog.spitzenpfeil.org"
@@
 P 950 3200
 F 0 "DZ1" H 950 3300 50  0000 C CNN
-F 1 "BZX84C_5V6" H 950 3100 40  0000 C CNN
+F 1 "BZX84C_5V1" H 950 3100 40  0000 C CNN
 	1    950  3200
 	0    -1   -1   0

Commit message: Fooling around a bit.
Parts:
- DS1: value MBRS140T3G -> SS14L (40V, 1A)
Changed lines of the file:
@@
-EESchema Schematic File Version 2  date Tue 20 Nov 2012 04:58:50 PM CET
+EESchema Schematic File Version 2
 LIBS:my_parts
 LIBS:power
@@
 LIBS:valves
 LIBS:LED-Square_PT4115-cache
-EELAYER 27 0
+EELAYER 24 0
 EELAYER END
 $Descr User 8268 5846
@@
 Sheet 1 1
 Title "LED-Square PT4115"
-Date "20 nov 2012"
-Rev "1.0"
-Comp "2012 - blog.spitzenpfeil.org"
+Date "05 Mar 2014"
+Rev "1.1"
+Comp "2014 - blog.spitzenpfeil.org"
 Comment1 ""
 Comment2 ""
@@
 F 0 "DZ1" H 950 3300 50  0000 C CNN
 F 1 "BZX84C_5V1" H 950 3100 40  0000 C CNN
+F 2 "" H 950 3200 60  0001 C CNN
+F 3 "" H 950 3200 60  0001 C CNN
 	1    950  3200
 	0    -1   -1   0
@@
 F 0 "#PWR01" H 950 3450 30  0001 C CNN
 F 1 "GND" H 950 3380 30  0001 C CNN
+F 2 "" H 950 3450 60  0001 C CNN
+F 3 "" H 950 3450 60  0001 C CNN
 	1    950  3450
 	1    0    0    -1
@@
 F 0 "R2" V 1030 2650 50  0000 C CNN
 F 1 "1k" V 950 2650 50  0000 C CNN
+F 2 "" H 950 2650 60  0001 C CNN
+F 3 "" H 950 2650 60  0001 C CNN
 	1    950  2650
 	1    0    0    -1
@@
 F 0 "R1" V 2280 2700 50  0000 C CNN
 F 1 "1M" V 2200 2700 50  0000 C CNN
+F 2 "" H 2200 2700 60  0001 C CNN
+F 3 "" H 2200 2700 60  0001 C CNN
 	1    2200 2700
 	1    0    0    -1
@@
 F 0 "#PWR02" H 2000 3000 30  0001 C CNN
 F 1 "GND" H 2000 2930 30  0001 C CNN
+F 2 "" H 2000 3000 60  0001 C CNN
+F 3 "" H 2000 3000 60  0001 C CNN
 	1    2000 3000
 	1    0    0    -1
@@
 F 0 "C6" H 1850 2800 50  0000 L CNN
 F 1 "1.25µF/s" V 1600 2550 50  0000 L CNN
+F 2 "" H 1800 2700 60  0001 C CNN
+F 3 "" H 1800 2700 60  0001 C CNN
 	1    1800 2700
 	1    0    0    -1
@@
 F 0 "#PWR03" H 5750 900 30  0001 C CNN
 F 1 "VCC" H 5750 900 30  0000 C CNN
+F 2 "" H 5750 800 60  0001 C CNN
+F 3 "" H 5750 800 60  0001 C CNN
 	1    5750 800
 	1    0    0    -1
@@
 F 0 "#PWR04" H 5750 1500 30  0001 C CNN
 F 1 "GND" H 5750 1430 30  0001 C CNN
+F 2 "" H 5750 1500 60  0001 C CNN
+F 3 "" H 5750 1500 60  0001 C CNN
 	1    5750 1500
 	1    0    0    -1
@@
 F 0 "C5" H 6550 1250 50  0000 L CNN
 F 1 "10µF" H 6550 1050 50  0000 L CNN
+F 2 "" H 6500 1150 60  0001 C CNN
+F 3 "" H 6500 1150 60  0001 C CNN
 	1    6500 1150
 	1    0    0    -1
@@
 F 0 "C4" H 6300 1250 50  0000 L CNN
 F 1 "10µF" H 6300 1050 50  0000 L CNN
+F 2 "" H 6250 1150 60  0001 C CNN
+F 3 "" H 6250 1150 60  0001 C CNN
 	1    6250 1150
 	1    0    0    -1
@@
 F 0 "C3" H 6050 1250 50  0000 L CNN
 F 1 "10µF" H 6050 1050 50  0000 L CNN
+F 2 "" H 6000 1150 60  0001 C CNN
+F 3 "" H 6000 1150 60  0001 C CNN
 	1    6000 1150
 	1    0    0    -1
@@
 F 0 "C2" H 5800 1250 50  0000 L CNN
 F 1 "10µF" H 5800 1050 50  0000 L CNN
+F 2 "" H 5750 1150 60  0001 C CNN
+F 3 "" H 5750 1150 60  0001 C CNN
 	1    5750 1150
 	1    0    0    -1
@@
 F 0 "#PWR05" H 7100 2200 30  0001 C CNN
 F 1 "VCC" H 7100 2200 30  0000 C CNN
+F 2 "" H 7100 2100 60  0001 C CNN
+F 3 "" H 7100 2100 60  0001 C CNN
 	1    7100 2100
 	-1   0    0    1
@@
 F 0 "#PWR06" H 5600 2200 30  0001 C CNN
 F 1 "VCC" H 5600 2200 30  0000 C CNN
+F 2 "" H 5600 2100 60  0001 C CNN
+F 3 "" H 5600 2100 60  0001 C CNN
 	1    5600 2100
 	-1   0    0    1
@@
 F 0 "#PWR07" H 7100 1900 30  0001 C CNN
 F 1 "GND" H 7100 1830 30  0001 C CNN
+F 2 "" H 7100 1900 60  0001 C CNN
+F 3 "" H 7100 1900 60  0001 C CNN
 	1    7100 1900
 	1    0    0    -1
@@
 F 0 "#PWR08" H 5600 1900 30  0001 C CNN
 F 1 "GND" H 5600 1830 30  0001 C CNN
+F 2 "" H 5600 1900 60  0001 C CNN
+F 3 "" H 5600 1900 60  0001 C CNN
 	1    5600 1900
 	1    0    0    -1
@@
 F 0 "P2" V 6450 2100 60  0000 C CNN
 F 1 "OUT" V 6550 2100 60  0000 C CNN
+F 2 "" H 6500 2100 60  0001 C CNN
+F 3 "" H 6500 2100 60  0001 C CNN
 	1    6500 2100
 	-1   0    0    1
@@
 F 0 "P1" V 6150 2100 60  0000 C CNN
 F 1 "IN" V 6250 2100 60  0000 C CNN
+F 2 "" H 6200 2100 60  0001 C CNN
+F 3 "" H 6200 2100 60  0001 C CNN
 	1    6200 2100
 	1    0    0    -1
@@
 F 0 "MH4" H 5780 2950 40  0000 L CNN
 F 1 "CONN_1" H 5700 3005 30  0001 C CNN
+F 2 "" H 5700 2950 60  0001 C CNN
+F 3 "" H 5700 2950 60  0001 C CNN
 	1    5700 2950
 	1    0    0    -1
@@
 F 0 "MH3" H 5780 2850 40  0000 L CNN
 F 1 "CONN_1" H 5700 2905 30  0001 C CNN
+F 2 "" H 5700 2850 60  0001 C CNN
+F 3 "" H 5700 2850 60  0001 C CNN
 	1    5700 2850
 	1    0    0    -1
@@
 F 0 "MH2" H 5780 2750 40  0000 L CNN
 F 1 "CONN_1" H 5700 2805 30  0001 C CNN
+F 2 "" H 5700 2750 60  0001 C CNN
+F 3 "" H 5700 2750 60  0001 C CNN
 	1    5700 2750
 	1    0    0    -1
@@
 F 0 "MH1" H 5780 2650 40  0000 L CNN
 F 1 "CONN_1" H 5700 2705 30  0001 C CNN
+F 2 "" H 5700 2650 60  0001 C CNN
+F 3 "" H 5700 2650 60  0001 C CNN
 	1    5700 2650
 	1    0    0    -1
@@
 F 0 "#PWR09" H 7400 1400 30  0001 C CNN
 F 1 "VCC" H 7400 1400 30  0000 C CNN
+F 2 "" H 7400 1300 60  0001 C CNN
+F 3 "" H 7400 1300 60  0001 C CNN
 	1    7400 1300
 	-1   0    0    1
@@
 F 0 "#PWR010" H 7100 1300 30  0001 C CNN
 F 1 "GND" H 7100 1230 30  0001 C CNN
+F 2 "" H 7100 1300 60  0001 C CNN
+F 3 "" H 7100 1300 60  0001 C CNN
 	1    7100 1300
 	1    0    0    -1
@@
 F 0 "#FLG011" H 7400 1245 30  0001 C CNN
 F 1 "PWR_FLAG" H 7400 1330 30  0000 C CNN
+F 2 "" H 7400 1150 60  0001 C CNN
+F 3 "" H 7400 1150 60  0001 C CNN
 	1    7400 1150
 	1    0    0    -1
@@
 F 0 "#FLG012" H 7100 1245 30  0001 C CNN
 F 1 "PWR_FLAG" H 7100 1330 30  0000 C CNN
+F 2 "" H 7100 1150 60  0001 C CNN
+F 3 "" H 7100 1150 60  0001 C CNN
 	1    7100 1150
 	1    0    0    -1
@@
 F 0 "#PWR013" H 2950 1950 30  0001 C CNN
 F 1 "VCC" H 2950 1950 30  0000 C CNN
+F 2 "" H 2950 1850 60  0001 C CNN
+F 3 "" H 2950 1850 60  0001 C CNN
 	1    2950 1850
 	1    0    0    -1
@@
 F 0 "#PWR014" H 800 1150 30  0001 C CNN
 F 1 "VCC" H 800 1150 30  0000 C CNN
+F 2 "" H 800 1050 60  0001 C CNN
+F 3 "" H 800 1050 60  0001 C CNN
 	1    800  1050
 	1    0    0    -1
@@
 F 0 "#PWR015" H 800 1700 30  0001 C CNN
 F 1 "GND" H 800 1630 30  0001 C CNN
+F 2 "" H 800 1700 60  0001 C CNN
+F 3 "" H 800 1700 60  0001 C CNN
 	1    800  1700
 	1    0    0    -1
@@
 F 0 "#PWR016" H 2400 1400 30  0001 C CNN
 F 1 "VCC" H 2400 1400 30  0000 C CNN
+F 2 "" H 2400 1300 60  0001 C CNN
+F 3 "" H 2400 1300 60  0001 C CNN
 	1    2400 1300
 	1    0    0    -1
@@
 F 0 "#PWR017" H 1200 1700 30  0001 C CNN
 F 1 "GND" H 1200 1630 30  0001 C CNN
+F 2 "" H 1200 1700 60  0001 C CNN
+F 3 "" H 1200 1700 60  0001 C CNN
 	1    1200 1700
 	1    0    0    -1
@@
 F 0 "D4" H 4100 1250 50  0000 C CNN
 F 1 "LED" H 4100 1050 50  0000 C CNN
+F 2 "" H 4100 1150 60  0001 C CNN
+F 3 "" H 4100 1150 60  0001 C CNN
 	1    4100 1150
 	0    1    1    0
@@
 F 0 "D6" H 4700 1250 50  0000 C CNN
 F 1 "LED" H 4700 1050 50  0000 C CNN
+F 2 "" H 4700 1150 60  0001 C CNN
+F 3 "" H 4700 1150 60  0001 C CNN
 	1    4700 1150
 	0    1    1    0
@@
 F 0 "D5" H 4400 1250 50  0000 C CNN
 F 1 "LED" H 4400 1050 50  0000 C CNN
+F 2 "" H 4400 1150 60  0001 C CNN
+F 3 "" H 4400 1150 60  0001 C CNN
 	1    4400 1150
 	0    -1   -1   0
@@
 F 0 "D3" H 3800 1250 50  0000 C CNN
 F 1 "LED" H 3800 1050 50  0000 C CNN
+F 2 "" H 3800 1150 60  0001 C CNN
+F 3 "" H 3800 1150 60  0001 C CNN
 	1    3800 1150
 	0    -1   -1   0
@@
 F 0 "D2" H 3500 1250 50  0000 C CNN
 F 1 "LED" H 3500 1050 50  0000 C CNN
+F 2 "" H 3500 1150 60  0001 C CNN
+F 3 "" H 3500 1150 60  0001 C CNN
 	1    3500 1150
 	0    1    1    0
@@
 F 0 "D1" H 3200 1250 50  0000 C CNN
 F 1 "LED" H 3200 1050 50  0000 C CNN
+F 2 "" H 3200 1150 60  0001 C CNN
+F 3 "" H 3200 1150 60  0001 C CNN
 	1    3200 1150
 	0    -1   -1   0
@@
 F 0 "C1" H 850 1500 50  0000 L CNN
 F 1 "10µF" H 850 1300 50  0000 L CNN
+F 2 "" H 800 1400 60  0001 C CNN
+F 3 "" H 800 1400 60  0001 C CNN
 	1    800  1400
 	1    0    0    -1
@@
 P 2550 1900
 F 0 "DS1" H 2550 2000 40  0000 C CNN
-F 1 "MBRS140T3G" H 2550 1800 40  0000 C CNN
+F 1 "SS14L (40V, 1A)" H 2550 1800 40  0000 C CNN
+F 2 "" H 2550 1900 60  0001 C CNN
+F 3 "" H 2550 1900 60  0001 C CNN
 	1    2550 1900
 	1    0    0    -1
@@
 F 0 "R_CS1" V 2750 1350 50  0000 C CNN
 F 1 "1R" V 2650 1350 50  0000 C CNN
+F 2 "" H 2650 1350 60  0001 C CNN
+F 3 "" H 2650 1350 60  0001 C CNN
 	1    2650 1350
 	0    -1   -1   0
@@
 F 0 "L1" V 2600 1650 40  0000 C CNN
 F 1 "100µH" V 2750 1650 40  0000 C CNN
+F 2 "" H 2650 1650 60  0001 C CNN
+F 3 "" H 2650 1650 60  0001 C CNN
 	1    2650 1650
 	0    -1   -1   0
@@
 F 0 "U1" H 1700 1150 60  0000 C CNN
 F 1 "PT4115-SOT89-5" H 1700 1750 60  0000 C CNN
+F 2 "" H 1700 1450 60  0001 C CNN
+F 3 "" H 1700 1450 60  0001 C CNN
 	1    1700 1450
 	1    0    0    -1

Commit message: R_CS --> 1206. Couldn't get 1R1 in 0805.
Parts:
- added R_CS2: 1R1, symbol R
- R_CS1: value 1R -> 1R1
Connections:
- net CSN: now also R_CS2.2
- net VCC: now also R_CS2.1
Other:
- moved on the sheet: R_CS1
Changed lines of the file:
@@
 Title "LED-Square PT4115"
 Date "05 Mar 2014"
-Rev "1.1"
+Rev "1.11"
 Comp "2014 - blog.spitzenpfeil.org"
 Comment1 ""
@@
 	800  1600 800  1700
 Wire Wire Line
-	2950 1350 2950 1450
+	2950 1250 2950 1450
 Wire Wire Line
 	2950 1450 2150 1450
@@
 	4700 900  4700 950
 Wire Wire Line
-	2150 1350 2400 1350
-Wire Wire Line
-	2400 1350 2400 1300
+	2400 1350 2150 1350
+Wire Wire Line
+	2400 1200 2400 1350
 Wire Wire Line
 	800  1050 800  1200
@@
 Text Label 2250 1900 2    60   ~ 0
 SW
-Text Notes 2300 1150 0    60   ~ 0
+Text Notes 2300 1050 0    60   ~ 0
 (24V)
 Text Notes 3700 750  0    60   ~ 0
@@
 L VCC #PWR016
 U 1 1 506F3A0F
-P 2400 1300
-F 0 "#PWR016" H 2400 1400 30  0001 C CNN
-F 1 "VCC" H 2400 1400 30  0000 C CNN
-F 2 "" H 2400 1300 60  0001 C CNN
-F 3 "" H 2400 1300 60  0001 C CNN
-	1    2400 1300
+P 2400 1200
+F 0 "#PWR016" H 2400 1300 30  0001 C CNN
+F 1 "VCC" H 2400 1300 30  0000 C CNN
+F 2 "" H 2400 1200 60  0001 C CNN
+F 3 "" H 2400 1200 60  0001 C CNN
+	1    2400 1200
 	1    0    0    -1
 $EndComp
@@
 L R R_CS1
 U 1 1 506F3496
-P 2650 1350
-F 0 "R_CS1" V 2750 1350 50  0000 C CNN
-F 1 "1R" V 2650 1350 50  0000 C CNN
-F 2 "" H 2650 1350 60  0001 C CNN
-F 3 "" H 2650 1350 60  0001 C CNN
-	1    2650 1350
+P 2650 1250
+F 0 "R_CS1" V 2750 1250 50  0000 C CNN
+F 1 "1R1" V 2650 1250 50  0000 C CNN
+F 2 "" H 2650 1250 60  0001 C CNN
+F 3 "" H 2650 1250 60  0001 C CNN
+	1    2650 1250
 	0    -1   -1   0
 $EndComp
@@
 Text Notes 550  5100 0    60   ~ 0
 (*) Don't use C6 when driving DIM with a 5V PWM signal.\n    Replace R1 with a 10k pull-down resistor.
+$Comp
+L R R_CS2
+U 1 1 531746E7
+P 2650 1350
+F 0 "R_CS2" V 2600 1350 50  0001 C CNN
+F 1 "1R1" V 2650 1350 50  0000 C CNN
+F 2 "" H 2650 1350 60  0001 C CNN
+F 3 "" H 2650 1350 60  0001 C CNN
+	1    2650 1350
+	0    -1   -1   0
+$EndComp
+Wire Wire Line
+	2900 1250 2950 1250
+Connection ~ 2400 1250
 $EndSCHEMATC

Commit message: Now using 2 pins for the DIM signal as well.
Connections:
- net DIM: now also P1.5, P2.2
- no-connect marks 6 -> 4
Changed lines of the file:
@@
 Sheet 1 1
 Title "LED-Square PT4115"
-Date "05 Mar 2014"
-Rev "1.11"
+Date "13 Sep 2014"
+Rev "1.2"
 Comp "2014 - blog.spitzenpfeil.org"
 Comment1 ""
@@
 	1    0    0    -1
 $EndComp
-NoConn ~ 6850 2250
-NoConn ~ 5850 2250
 Text Label 6950 2350 0    60   ~ 0
 DIM
@@
 	2900 1250 2950 1250
 Connection ~ 2400 1250
+Wire Wire Line
+	6850 2250 6900 2250
+Wire Wire Line
+	6900 2250 6900 2350
+Connection ~ 6900 2350
+Wire Wire Line
+	5800 2350 5800 2250
+Wire Wire Line
+	5800 2250 5850 2250
+Connection ~ 5800 2350
 $EndSCHEMATC
